File: output/pcbs/nib.kicad_pcb (KiCad board)
At the start: 2 copper layers, 152.8 x 120 mm, 75 parts, among them J1 Jumper

Commit message: need to fix data/clock still
Parts:
- moved J1 4.90 mm to (213.6, 79.0)
- moved DISP2 2.50 mm to (210.6, 83.0)
- moved DISP3 1.30 mm to (210.6, 85.0)
- moved B1 0.10 mm to (218.6, 80.8)
- moved DISP1 0.10 mm to (208.6, 90.0)
- moved SW1 0.10 mm to (218.6, 90.0)
Connections:
- net RESET renamed TPR
Other:
- outline, holes or cut-outs redrawn
Changed lines of the file:
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@@
 (net 5 "DATA")
 (net 6 "CLK")
-(net 7 "RESET")
+(net 7 "TPR")
 (net 8 "R0")
 (net 9 "R1")
@@
 (add_net "DATA")
 (add_net "CLK")
-(add_net "RESET")
+(add_net "TPR")
 (add_net "R0")
 (add_net "R1")
@@
           (pad 7 thru_hole circle (at 7.62 2.540000000000001) (size 1.7 1.7) (drill 1) (layers *.Cu *.Mask) (net 36 "MCU1_7"))
           (pad 118 thru_hole circle (at -3.262 2.540000000000001) (size 0.8 0.8) (drill 0.4) (layers *.Cu *.Mask) (net 17 "C2"))
-          (pad 7 thru_hole circle (at 3.262 2.540000000000001) (size 0.8 0.8) (drill 0.4) (layers *.Cu *.Mask) (net 7 "RESET"))
+          (pad 7 thru_hole circle (at 3.262 2.540000000000001) (size 0.8 0.8) (drill 0.4) (layers *.Cu *.Mask) (net 7 "TPR"))
           (pad 18 smd custom (at -5.5 2.540000000000001) (size 0.2 0.2) (layers F.Cu F.Mask) (net 35 "MCU1_18")
             (zone_connect 2)
@@
             ) (width 0))
           ))
-          (pad 7 smd custom (at 4.775 2.540000000000001 180) (size 0.2 0.2) (layers F.Cu F.Mask) (net 7 "RESET")
+          (pad 7 smd custom (at 4.775 2.540000000000001 180) (size 0.2 0.2) (layers F.Cu F.Mask) (net 7 "TPR")
             (zone_connect 2)
             (options (clearance outline) (anchor rect))
@@
             ) (width 0))
           ))
-          (pad 7 smd custom (at -4.775 2.540000000000001) (size 0.2 0.2) (layers B.Cu B.Mask) (net 7 "RESET")
+          (pad 7 smd custom (at -4.775 2.540000000000001) (size 0.2 0.2) (layers B.Cu B.Mask) (net 7 "TPR")
             (zone_connect 2)
             (options (clearance outline) (anchor rect))
@@
             ) (width 0))
           ))
-            (fp_text user RESET (at -3 2.540000000000001) (layer F.SilkS)
+            (fp_text user TPR (at -3 2.540000000000001) (layer F.SilkS)
               (effects (font (size 1 1) (thickness 0.15)) (justify left))
             )
@@
               (effects (font (size 1 1) (thickness 0.15)) (justify right mirror))
             )
-            (fp_text user RESET (at 3 2.540000000000001 180) (layer B.SilkS)
+            (fp_text user TPR (at 3 2.540000000000001 180) (layer B.SilkS)
               (effects (font (size 1 1) (thickness 0.15)) (justify left mirror))
             )
@@
               (effects (font (size 0.5 0.5) (thickness 0.08)))
             )
-            (fp_text user RESET (at 3.262 1.7400000000000002) (layer F.Fab)
+            (fp_text user TPR (at 3.262 1.7400000000000002) (layer F.Fab)
               (effects (font (size 0.5 0.5) (thickness 0.08)))
             )
@@
               (effects (font (size 0.5 0.5) (thickness 0.08)) (justify mirror))
             )
-            (fp_text user RESET (at 3.262 1.7400000000000002 180) (layer B.Fab)
+            (fp_text user TPR (at 3.262 1.7400000000000002 180) (layer B.Fab)
               (effects (font (size 0.5 0.5) (thickness 0.08)) (justify mirror))
             )
@@
     )
         (module power_switch (layer F.Cu)
-          (at 218.675 89.95 0)
+          (at 218.57500000000002 89.95 0)
           (attr smd)
           (fp_text reference "SW1" (at -3.6 0 -90) (layer F.SilkS) hide
@@
         (descr "Two pin through hole Tactile Switch, the same as on the Corne")
         (tags "Tactile Switch")
-        (at 218.65 80.8 -90)
+        (at 218.55 80.8 -90)
         (fp_text reference "B1" (at 0 2.55) (layer F.SilkS) hide (effects (font (size 1 1) (thickness 0.15))))
         (fp_text value "" (at 0 -2.55) (layer F.Fab) (effects (font (size 1 1) (thickness 0.15))))
@@
         )
 (module HRS_FH34SRJ-8S-0.5SH_50_ (layer F.Cu)
-        (at 208.675 89.95 0)
+        (at 208.57500000000002 89.95 0)
   (descr "")
   (attr smd)
@@
 )
     (module RES_ERJ2RKF4701X (layer F.Cu)
-        (at 208.07500000000002 82.95 0)
+        (at 210.57500000000002 82.95 0)
   (descr "")
   (attr smd)
@@
 )
     (module RES_ERJ2RKF4701X (layer F.Cu)
-        (at 209.275 84.95 0)
+        (at 210.57500000000002 84.95 0)
   (descr "")
   (attr smd)
@@
 )
         (module lib:Jumper (layer F.Cu)
-        (at 208.675 78.95 90)
+        (at 213.57500000000002 78.95 90)
         (fp_text reference "J1" (at 0 0) (layer F.SilkS) hide (effects (font (size 1.27 1.27) (thickness 0.15))))
         (fp_text value Jumper (at 0 -7.3) (layer F.Fab) (effects (font (size 1 1) (thickness 0.15))))
@@
         (clearance 0.1905) (net 79 "RESETC"))
         (pad 2 smd rect (at 0.50038 0 90) (size 0.635 1.143) (layers F.Cu F.Paste F.Mask)
-        (clearance 0.1905) (net 7 "RESET")))
+        (clearance 0.1905) (net 7 "TPR")))
       (module trackpoint_mount_t430 (layer F.Cu)
         (at 181 88.5 45)
@@
 (gr_line (start 199 37.5) (end 182 37.5) (angle 90) (layer Edge.Cuts) (width 0.15))
 (gr_arc (start 199 38.5) (end 200 38.5) (angle -90) (layer Edge.Cuts) (width 0.15))
+(gr_circle (center 109 41.35) (end 110.1 41.35) (layer Edge.Cuts) (width 0.15))
+(gr_circle (center 121.6 111) (end 122.69999999999999 111) (layer Edge.Cuts) (width 0.15))
+(gr_circle (center 200.26 41.39) (end 201.35999999999999 41.39) (layer Edge.Cuts) (width 0.15))
+(gr_circle (center 226.59641939999997 109.05874539999999) (end 227.69641939999997 109.05874539999999) (layer Edge.Cuts) (width 0.15))
 )
